File: podlewacz/untitled 3.sch (EAGLE design)
At the start: 17 parts

Commit message: usb asp adapter
Parts:
- removed PIN_IN: (no value), con-lstb:MA08-1
- added BATTERY: PINHEAD-1X2, mcp73831:PINHEAD-1X2
- added M1_LED, M2-LED, M3-LED, M4-LED: green, led:LEDCHIP-LED0805
- added PROMINI-DOWN: (no value), con-lsta:FE05-1
- added PROMINI-LEFT, PROMINI-RIGHT: (no value), con-lsta:FE12-1
- added PROMINI-UP: (no value), con-lsta:FE06-1
- added R10, R11, R7, R8, R9: 510r, resistor:R-EU_M0805
- added R12: 10k, resistor:R-EU_R1206
- added S1: DTSM-3, switch-tact:DTSM-3
- added WARNING: red, led:LEDCHIP-LED0805
Connections:
- new net LED-GREEN-1: PROMINI-LEFT.12, R7.1
- new net LED-GREEN-2: PROMINI-LEFT.11, R8.1
- new net LED-GREEN-3: PROMINI-LEFT.8, R9.1
- new net LED-GREEN-4: PROMINI-LEFT.7, R10.1
- new net LED-RED: PROMINI-LEFT.6, R11.1
- new net N$4: R11.2, WARNING.A
- new net N$5: M4-LED.A, R10.2
- new net N$6: M3-LED.A, R9.2
- new net N$7: M2-LED.A, R8.2
- new net N$8: M1_LED.A, R7.2
- new net OPTIONS: PROMINI-LEFT.5, R12.1, S1.2
- net +5V: now also PROMINI-RIGHT.1, S1.1; no longer PIN_IN.8
- net GND: now also BATTERY.2, M1_LED.C, M2-LED.C, M3-LED.C, M4-LED.C, PROMINI-DOWN.1, PROMINI-LEFT.4, PROMINI-RIGHT.2, R12.2, WARNING.C; no longer PIN_IN.2, PIN_IN.5
- net M1_IN: now also PROMINI-DOWN.2; no longer PIN_IN.6
- net M2_IN: now also PROMINI-DOWN.3; no longer PIN_IN.7
- net M3_IN: now also PROMINI-RIGHT.6; no longer PIN_IN.3
- net M4_IN: now also PROMINI-RIGHT.5; no longer PIN_IN.4
- net VCC: now also BATTERY.1; no longer PIN_IN.1
