File: test/untitled.brd (EAGLE design)
At the start: 14.2 x 30.7 mm, 0 parts

Commit message: 3.7 protect
Parts:
- added IC1, IC2: 4051D, 40xx:SO16
Connections:
- new net GND: IC1.8, IC2.8
- new net VCC: IC1.16, IC2.16
- new net VEE: IC1.7, IC2.7
Changed lines of the file:
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@@
 <?xml version="1.0" encoding="utf-8"?>
 <!DOCTYPE eagle SYSTEM "eagle.dtd">
-<eagle version="7.4.0">
+<eagle version="7.5.0">
 <drawing>
 <settings>
@@
 <layer number="51" name="tDocu" color="7" fill="1" visible="yes" active="yes"/>
 <layer number="52" name="bDocu" color="7" fill="1" visible="yes" active="yes"/>
+<layer number="91" name="Nets" color="2" fill="1" visible="no" active="no"/>
+<layer number="92" name="Busses" color="1" fill="1" visible="no" active="no"/>
+<layer number="93" name="Pins" color="2" fill="1" visible="no" active="no"/>
+<layer number="94" name="Symbols" color="4" fill="1" visible="no" active="no"/>
+<layer number="95" name="Names" color="7" fill="1" visible="no" active="no"/>
+<layer number="96" name="Values" color="7" fill="1" visible="no" active="no"/>
+<layer number="97" name="Info" color="7" fill="1" visible="no" active="no"/>
+<layer number="98" name="Guide" color="6" fill="1" visible="no" active="no"/>
 <layer number="100" name="descripion" color="0" fill="1" visible="yes" active="yes"/>
 </layers>
@@
 </autorouter>
 <elements>
+<element name="IC1" library="40xx" package="SO16" value="4051D" x="5.2832" y="-36.576"/>
+<element name="IC2" library="40xx" package="SO16" value="4051D" x="5.2832" y="-45.212"/>
 </elements>
 <signals>
@@
 <wire x1="5.1816" y1="-3.4036" x2="5.1816" y2="-2.794" width="0.0508" layer="1"/>
 </signal>
+<signal name="VEE">
+<contactref element="IC1" pad="7"/>
+<contactref element="IC2" pad="7"/>
+<wire x1="8.4582" y1="-39.6494" x2="8.4582" y2="-48.2854" width="0" layer="19" extent="1-1"/>
+</signal>
+<signal name="GND">
+<contactref element="IC1" pad="8"/>
+<contactref element="IC2" pad="8"/>
+<wire x1="9.7282" y1="-39.6494" x2="9.7282" y2="-48.2854" width="0" layer="19" extent="1-1"/>
+</signal>
+<signal name="VCC">
+<contactref element="IC1" pad="16"/>
+<contactref element="IC2" pad="16"/>
+<wire x1="0.8382" y1="-33.5026" x2="0.8382" y2="-42.1386" width="0" layer="19" extent="1-1"/>
+</signal>
 </signals>
