File: usb asp adapter/untitled.brd (EAGLE design)
At the start: 19.2 x 31.5 mm, 3 parts

Commit message: 3.7 protect
Connections:
- net VCC: now also PROMINI-RIGHT.1, SV1.1; no longer PROMINI-RIGHT.4, SV1.4
Routing:
- net VCC: track 15.8 -> 21.3 mm
- net RST: track 25.2 -> 20.5 mm
Other:
- board size 19.2 x 31.5 mm -> 18.5 x 31.5 mm
- board text removed: "RAW"
Changed lines of the file:
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@@
 <board>
 <plain>
-<wire x1="7.62" y1="12.446" x2="26.848" y2="12.446" width="0" layer="20"/>
-<wire x1="26.848" y1="12.446" x2="26.848" y2="43.932" width="0" layer="20"/>
-<wire x1="26.848" y1="43.932" x2="7.62" y2="43.932" width="0" layer="20"/>
+<wire x1="7.62" y1="12.446" x2="26.086" y2="12.446" width="0" layer="20"/>
+<wire x1="26.086" y1="12.446" x2="26.086" y2="43.932" width="0" layer="20"/>
+<wire x1="26.086" y1="43.932" x2="7.62" y2="43.932" width="0" layer="20"/>
 <wire x1="7.62" y1="43.932" x2="7.62" y2="12.446" width="0" layer="20"/>
-<text x="20.828" y="41.529" size="0.8128" layer="16" font="vector" ratio="20" rot="MR0">RAW</text>
-<text x="20.828" y="38.989" size="0.8128" layer="16" font="vector" ratio="20" rot="MR0">GND</text>
+<text x="21.336" y="38.989" size="0.8128" layer="16" font="vector" ratio="20" rot="MR0">GND</text>
 <text x="19.812" y="13.589" size="0.8128" layer="16" font="vector" ratio="20" rot="MR0">10</text>
 <rectangle x1="18.542" y1="27.432" x2="19.304" y2="30.988" layer="42"/>
 <text x="12.7" y="24.638" size="1.27" layer="16" font="vector" ratio="20" rot="MR90">PROMINI</text>
-<text x="25.908" y="16.764" size="0.8128" layer="16" font="vector" ratio="20" rot="MR270" align="bottom-center">usbasp
+<text x="25.4" y="16.51" size="0.8128" layer="16" font="vector" ratio="20" rot="MR270" align="bottom-center">usbasp
 adapter
 by Sh4DoV</text>
@@
 <signal name="VCC">
 <contactref element="USB-ASP" pad="2"/>
-<contactref element="PROMINI-RIGHT" pad="4"/>
-<contactref element="SV1" pad="4"/>
-<wire x1="10.16" y1="34.29" x2="16.51" y2="34.29" width="0.4064" layer="16"/>
-<wire x1="24.13" y1="34.29" x2="24.13" y2="35.306" width="0.4064" layer="16"/>
-<wire x1="24.13" y1="35.306" x2="23.622" y2="35.814" width="0.4064" layer="16"/>
-<wire x1="23.622" y1="35.814" x2="20.574" y2="35.814" width="0.4064" layer="16"/>
-<wire x1="20.574" y1="35.814" x2="19.05" y2="34.29" width="0.4064" layer="16"/>
-<wire x1="19.05" y1="34.29" x2="16.51" y2="34.29" width="0.4064" layer="16"/>
+<contactref element="PROMINI-RIGHT" pad="1"/>
+<contactref element="SV1" pad="1"/>
+<wire x1="10.16" y1="41.91" x2="16.51" y2="41.91" width="0.4064" layer="16"/>
+<wire x1="24.13" y1="34.29" x2="24.13" y2="41.402" width="0.4064" layer="16"/>
+<wire x1="24.13" y1="41.402" x2="23.622" y2="41.91" width="0.4064" layer="16"/>
+<wire x1="23.622" y1="41.91" x2="16.51" y2="41.91" width="0.4064" layer="16"/>
 </signal>
 <signal name="MOSI">
@@
 <contactref element="SV1" pad="3"/>
 <wire x1="10.16" y1="36.83" x2="16.51" y2="36.83" width="0.4064" layer="16"/>
-<wire x1="16.51" y1="36.83" x2="24.13" y2="36.83" width="0.4064" layer="16"/>
-<wire x1="24.13" y1="36.83" x2="25.654" y2="35.306" width="0.4064" layer="16"/>
-<wire x1="25.654" y1="35.306" x2="25.654" y2="30.988" width="0.4064" layer="16"/>
-<wire x1="25.654" y1="30.988" x2="25.146" y2="30.48" width="0.4064" layer="16"/>
-<wire x1="25.146" y1="30.48" x2="22.86" y2="30.48" width="0.4064" layer="16"/>
+<wire x1="16.51" y1="36.83" x2="22.352" y2="36.83" width="0.4064" layer="16"/>
 <wire x1="22.86" y1="30.48" x2="21.59" y2="29.21" width="0.4064" layer="16"/>
+<wire x1="22.86" y1="30.48" x2="22.86" y2="36.322" width="0.4064" layer="16"/>
+<wire x1="22.86" y1="36.322" x2="22.352" y2="36.83" width="0.4064" layer="16"/>
 </signal>
 <signal name="SCK">
@@
 <contactref element="SV1" pad="2"/>
 <polygon width="0.4064" layer="16">
-<vertex x="6.096" y="9.652"/>
-<vertex x="31.75" y="9.652"/>
-<vertex x="31.75" y="46.482"/>
-<vertex x="6.096" y="46.482"/>
+<vertex x="7.112" y="11.938"/>
+<vertex x="26.416" y="11.938"/>
+<vertex x="26.416" y="44.45"/>
+<vertex x="7.112" y="44.45"/>
 </polygon>
 </signal>
@@
 </signal>
 <signal name="N$2">
-<polygon width="0.254" layer="16">
-<vertex x="6.858" y="44.45"/>
-<vertex x="27.686" y="44.45"/>
-<vertex x="27.686" y="11.684"/>
-<vertex x="6.858" y="11.684"/>
+<polygon width="0" layer="16">
+<vertex x="7.112" y="44.45"/>
+<vertex x="26.67" y="44.45"/>
+<vertex x="26.67" y="11.938"/>
+<vertex x="7.112" y="11.938"/>
 </polygon>
 </signal>
