File: usb asp adapter/untitled.sch (EAGLE design)
At the start: 3 parts

Commit message: 3.7 protect
Connections:
- net VCC: now also PROMINI-RIGHT.1, SV1.1; no longer PROMINI-RIGHT.4, SV1.4
Changed lines of the file:
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@@
 </segment>
 <segment>
-<pinref part="PROMINI-RIGHT" gate="G$1" pin="4"/>
-<wire x1="43.18" y1="68.58" x2="45.72" y2="68.58" width="0.1524" layer="91"/>
-<label x="45.72" y="68.58" size="1.27" layer="95" xref="yes"/>
+<pinref part="PROMINI-RIGHT" gate="G$1" pin="1"/>
+<wire x1="43.18" y1="76.2" x2="45.72" y2="76.2" width="0.1524" layer="91"/>
+<label x="45.72" y="76.2" size="1.27" layer="95" xref="yes"/>
 </segment>
 <segment>
-<pinref part="SV1" gate="1" pin="4"/>
-<wire x1="20.32" y1="68.58" x2="22.86" y2="68.58" width="0.1524" layer="91"/>
-<label x="22.86" y="68.58" size="1.27" layer="95" xref="yes"/>
+<pinref part="SV1" gate="1" pin="1"/>
+<wire x1="20.32" y1="76.2" x2="22.86" y2="76.2" width="0.1524" layer="91"/>
+<label x="22.86" y="76.2" size="1.27" layer="95" xref="yes"/>
 </segment>
 </net>
