File: 3.7 protect/untitled.sch (EAGLE design)
At the start: 5 parts

Commit message: new update podlewacz v2
Parts:
- R1: value (none) -> 1k
Changed lines of the file:
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@@
 <part name="VIN" library="con-molex" deviceset="22-23-2021" device="" value=""/>
 <part name="VOUT" library="con-molex" deviceset="22-23-2021" device="" value=""/>
-<part name="R1" library="resistor" deviceset="R-EU_" device="R1206"/>
+<part name="R1" library="resistor" deviceset="R-EU_" device="R1206" value="1k"/>
 </parts>
 <sheets>
