File: capacitive measure sensor/untitled.brd (EAGLE design)
At the start: 10 x 85 mm, 0 parts

Commit message: gas sensor
Changed lines of the file:
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@@
 <?xml version="1.0" encoding="utf-8"?>
 <!DOCTYPE eagle SYSTEM "eagle.dtd">
-<eagle version="7.5.0">
+<eagle version="7.6.0">
 <drawing>
 <settings>
@@
 <setting verticaltext="up"/>
 </settings>
-<grid distance="50" unitdist="mil" unit="mil" style="dots" multiple="1" display="yes" altdistance="0.025" altunitdist="inch" altunit="inch"/>
+<grid distance="25" unitdist="mil" unit="mil" style="lines" multiple="1" display="yes" altdistance="0.025" altunitdist="inch" altunit="inch"/>
 <layers>
 <layer number="1" name="Top" color="4" fill="1" visible="yes" active="yes"/>
@@
 <dimension x1="0" y1="0" x2="0" y2="85" x3="-6" y3="42.5" textsize="1.778" layer="47"/>
 <dimension x1="0" y1="0" x2="10" y2="0" x3="5" y3="-4" textsize="1.778" layer="47"/>
-<wire x1="0" y1="0" x2="10" y2="0" width="0.4064" layer="20"/>
-<wire x1="10" y1="0" x2="10" y2="85" width="0.4064" layer="20"/>
-<wire x1="10" y1="85" x2="0" y2="85" width="0.4064" layer="20"/>
-<wire x1="0" y1="85" x2="0" y2="0" width="0.4064" layer="20"/>
-<polygon width="0" layer="17">
-<vertex x="3" y="2"/>
-<vertex x="4" y="2"/>
-<vertex x="4" y="1"/>
-<vertex x="3" y="1"/>
-</polygon>
-<polygon width="0" layer="17">
-<vertex x="7" y="2"/>
-<vertex x="6" y="2"/>
-<vertex x="6" y="1"/>
-<vertex x="7" y="1"/>
-</polygon>
+<wire x1="0" y1="0" x2="10" y2="0" width="0.127" layer="20"/>
+<wire x1="10" y1="0" x2="10" y2="85" width="0.127" layer="20"/>
+<wire x1="10" y1="85" x2="0" y2="85" width="0.127" layer="20"/>
+<wire x1="0" y1="85" x2="0" y2="0" width="0.127" layer="20"/>
 <polygon width="0" layer="17">
 <vertex x="1.27" y="3.81"/>
@@
 <vertex x="8.89" y="83.82"/>
 </polygon>
-<wire x1="8.89" y1="83.82" x2="8.89" y2="1.27" width="0.4064" layer="17"/>
-<wire x1="8.89" y1="1.27" x2="6.35" y2="1.27" width="0.4064" layer="17"/>
-<wire x1="3.81" y1="1.27" x2="1.27" y2="1.27" width="0.4064" layer="17"/>
-<wire x1="1.27" y1="1.27" x2="1.27" y2="78.74" width="0.4064" layer="17"/>
-<wire x1="1.27" y1="80.01" x2="1.27" y2="83.82" width="0.4064" layer="17"/>
+<wire x1="8.89" y1="83.6168" x2="8.89" y2="1.27" width="0.4064" layer="17"/>
+<wire x1="8.89" y1="1.27" x2="7.85" y2="1.27" width="0.4064" layer="17"/>
+<wire x1="2.183" y1="1.27" x2="1.27" y2="1.27" width="0.4064" layer="17"/>
+<wire x1="1.27" y1="1.27" x2="1.27" y2="78.5368" width="0.4064" layer="17"/>
+<wire x1="1.27" y1="80.2132" x2="1.27" y2="83.6168" width="0.4064" layer="17"/>
 </plain>
 <attributes>
@@
 </elements>
 <signals>
+<signal name="S$1">
+<via x="7" y="2" extent="1-16" drill="0.6" diameter="2.1844" shape="square"/>
+</signal>
+<signal name="S$2">
+<via x="3" y="2" extent="1-16" drill="0.6" diameter="2.1844" shape="square"/>
+</signal>
 </signals>
 </board>
