File: gas sensor/untitled.brd (EAGLE design)
At the start: 44 x 83.6 mm, 34 parts, among them J1 POWER_JACKPTH

Commit message: gas sensor
Parts:
- removed LED1: red, led:CHIPLED_0805
- removed LED2: green, led:CHIPLED_0805
- added GREEN_LED, RED_LED: (no value), con-headers-jp:SIP-100-02-32Y
- moved R6 2.50 mm to (28.7, 10.2)
- moved C5 2.50 mm to (31.0, 7.11)
- moved MCP73831 2.50 mm to (22.9, 9.91)
- moved R7 0.57 mm to (22.1, 6.35)
- moved R8 0.51 mm to (22.1, 3.56)
Connections:
- net CHARGE_GND: now also GREEN_LED.1; no longer LED2.C
- net CHARGE_VCC: now also RED_LED.2; no longer LED1.A
- net N$1: now also GREEN_LED.2; no longer LED2.A
- net N$15: now also RED_LED.1; no longer LED1.C
Routing:
- net CHARGE_GND: track 49.2 -> 56.7 mm
- net N$15: track 1.95 -> 5.28 mm
- net 3.7V_BAT: track 11.6 -> 14.4 mm
- net N$16: track 4.48 -> 7.27 mm
- net N$1: track 1.85 -> 4.29 mm
- net CHARGE_VCC: track 19.4 -> 17.9 mm
